File: Controller.kicad_sch (KiCad schematic)
At the start: 41 parts, among them J1 +5V, J2 Vmeas, J3 Vref, J4 Switch_Control, J5 Vofs, Q1 2N7002K, SW1 TVGP01-G73BB, U1 MCP1501-20E/CHY, U2 MCP4921-EP, U3 S-89713B-K8T2U, U4 MCP3421A0T-ECH, U7 ATMEGA328-PU_Arduino, U8 USB-C_to_Serial_Module, Y1 CSTLS16M0X55-B0

Commit message: Add BOM
Parts:
- removed J2: Vmeas, Connector_JST:JST_XH_B2B-XH-A_1x02_P2.50mm_Vertical, symbol Connector_Generic:Conn_01x02
- removed J3: Vref, Connector_JST:JST_XH_B2B-XH-A_1x02_P2.50mm_Vertical, symbol Connector_Generic:Conn_01x02
- removed J?: Thermister, Connector_JST:JST_XH_B2B-XH-A_1x02_P2.50mm_Vertical, symbol Connector_Generic:Conn_01x02
- removed R?: 1.5k, Resistor_THT:R_Axial_DIN0207_L6.3mm_D2.5mm_P10.16mm_Horizontal, symbol Device:R
- removed TP1: UART_RTS, TestPoint:TestPoint_Loop_D3.50mm_Drill0.9mm_Beaded, symbol Connector:TestPoint_Flag
- removed TP2: UART_TX, TestPoint:TestPoint_Loop_D3.50mm_Drill0.9mm_Beaded, symbol Connector:TestPoint_Flag
- removed TP3: UART_RX, TestPoint:TestPoint_Loop_D3.50mm_Drill0.9mm_Beaded, symbol Connector:TestPoint_Flag
- removed TP4: UART_CTS, TestPoint:TestPoint_Loop_D3.50mm_Drill0.9mm_Beaded, symbol Connector:TestPoint_Flag
- removed U1: MCP1501-20E/CHY, Package_TO_SOT_SMD:SOT-23-6, symbol Akizuki_PowerIC_Linear:Shunt_ConstV_6p
- removed U2: MCP4921-EP, Package_DIP:DIP-8_W7.62mm, symbol Analog_DAC:MCP4921-EP
- removed U7: ATMEGA328-PU_Arduino, digikey-footprints:DIP-28_W7.62mm, symbol Akizuki_MicrocontrollerBode:ATMEGA328-PU_Arduino
- removed U8: USB-C_to_Serial_Module, Akizuki_Module:USB-C_to_Serial_CH340E, symbol Akizuki_Modules:USB-C_to_Serial_Module
- removed Y1: CSTLS16M0X55-B0, Crystal:Resonator_Murata_CSTLSxxxG-3Pin_W8.0mm_H3.0mm, symbol Device:Resonator_Small
- added C1, C10, C11, C12, C14, C15, C19, C20, C21, C22, C23, C24, C4, C6, C7, C8, C9: 0.1u, Capacitor_SMD:C_0603_1608Metric, symbol Device:C_Small
- added C13: 1u, Capacitor_SMD:C_0603_1608Metric, symbol Device:C_Small
- added C25: 2.2u, Capacitor_SMD:C_0603_1608Metric, symbol Device:C_Small
- added C5: 10p, Capacitor_SMD:C_0603_1608Metric, symbol Device:C_Small
- added D2: LED, LED_SMD:LED_0603_1608Metric, symbol Device:LED
- added H1, H2, H3, H4: MountingHole, MountingHole:MountingHole_3.2mm_M3, symbol Mechanical:MountingHole
- added J1: Conn_01x16, Connector_PinSocket_2.54mm:PinSocket_1x16_P2.54mm_Vertical, symbol Connector_Generic:Conn_01x16
- added J2: USB_C_Receptacle_USB2.0_16P, Connector_USB:USB_C_Receptacle_GCT_USB4105-xx-A_16P_TopMnt_Horizontal, symbol Connector:USB_C_Receptacle_USB2.0_16P
- added J4: Conn_01x04, Connector_PinSocket_2.54mm:PinSocket_1x04_P2.54mm_Vertical, symbol Connector_Generic:Conn_01x04
- added J6: MOS_Thermister, Connector_JST:JST_XH_B2B-XH-A_1x02_P2.50mm_Vertical, symbol Connector_Generic:Conn_01x02
- added J8: AnalogIO, Connector_JST:JST_XH_B4B-XH-A_1x04_P2.50mm_Vertical, symbol Connector_Generic:Conn_01x04
- added JP1: 5VSW, Jumper:SolderJumper-2_P1.3mm_Open_TrianglePad1.0x1.5mm, symbol Jumper:SolderJumper_2_Open
- added JP2: GNDSW, Jumper:SolderJumper-2_P1.3mm_Open_TrianglePad1.0x1.5mm, symbol Jumper:SolderJumper_2_Open
- added P1: Eoshi-chan_Silk, Eoshi-chan:Eoshi-chan_logo_20x20, symbol Eoshi-chan:Eoshi-chan_Silk
- added Q1: 2N7002K, Package_TO_SOT_SMD:SOT-23, symbol Transistor_FET:2N7002K
- added R1: 5.1k, Resistor_SMD:R_0603_1608Metric, symbol Device:R
- added R15, R17, R18, R19, R2, R20, R21, R22, R23, R24, R25, R29, R33, R34, R35, R36, R40, R43, R44, R45, R8: 10k, Resistor_SMD:R_0603_1608Metric, symbol Device:R
- added R16, R31, R32: 100k, Resistor_SMD:R_0603_1608Metric, symbol Device:R
- added R26: 82, Resistor_SMD:R_0603_1608Metric, symbol Device:R
- added R30, R41: 3k, Resistor_SMD:R_0603_1608Metric, symbol Device:R
- added R4, R5: 27, Resistor_SMD:R_0603_1608Metric, symbol Device:R
- added R6: 470, Resistor_SMD:R_0603_1608Metric, symbol Device:R
- added R7: 1k, Resistor_SMD:R_0603_1608Metric, symbol Device:R
- added RV1, RV2, RV3, RV4: 10k, Potentiometer_THT:Potentiometer_Vishay_T73YP_Vertical, symbol Device:R_Potentiometer_Small
- added SW2: BOOTSEL, AM_Switch:TVBP06-B043Cx-B, symbol Switch:SW_Push
- added TP5: TP, TestPoint:TestPoint_THTPad_2.0x2.0mm_Drill1.0mm, symbol Connector:TestPoint_Probe
- added TP6, TP7, TP8: TestPoint_Probe, TestPoint:TestPoint_THTPad_2.0x2.0mm_Drill1.0mm, symbol Connector:TestPoint_Probe
- added U1: NJM2863, Package_TO_SOT_SMD:SOT-23-5, symbol Akizuki_PowerIC_Linear:NJM2863F33
- added U10, U11, U4, U9: S-89713B-K8T2U, Package_SO:MSOP-8_3x3mm_P0.65mm, symbol dk_Linear-Amplifiers-Instrumentation-OP-Amps-Buffer-Amps:LM358N_Obsolete
- added U2: RP2040, Package_DFN_QFN:QFN-56-1EP_7x7mm_P0.4mm_EP3.2x3.2mm, symbol MCU_RaspberryPi:RP2040
- added U3: W25Q16JVUXIQ, ROM:IC_W25Q16JVUXIQ_TR, symbol Memory_Flash:W25Q16JVSS
- added U5: MCP4725A0T-ECH, Package_TO_SOT_SMD:SOT-23-6, symbol Analog_DAC:MCP4725xxx-xCH
- added U8: NJM1431AU, Package_TO_SOT_SMD:SOT-89-3, symbol Akizuki_PowerIC_Linear:ShuntReg_3P
- added Y1: FA238V 12.000000MHz, Crystal:Crystal_SMD_SeikoEpson_FA238V-4Pin_3.2x2.5mm, symbol Device:Crystal_GND24
- C16: value 0.1u -> 1u; Akizuki_code (none) -> 116994
- C17: value 0.1u -> 10p; Akizuki_code (none) -> 113312
- C18, C3: Akizuki_code (none) -> 116143
- C2: value 2.2u -> 0.1u; Akizuki_code (none) -> 116143
- C26: renamed from C1; Akizuki_code (none) -> 116077
- D1: value BAT43 -> RB160M-30TR; footprint Diode_THT:D_DO-35_SOD27_P7.62mm_Horizontal -> Diode_SMD:D_SOD-123; Akizuki_code (none) -> 101398; now not fitted
- J5: value Vofs -> R_Thermister; Akizuki_code (none) -> 112247
- J7: renamed from J1; Akizuki_code (none) -> 112247
- J9: renamed from J4; Akizuki_code (none) -> 112250
- Q2: renamed from Q1; Akizuki_code (none) -> 104256
- R10: value 1k -> 10k; footprint Resistor_THT:R_Axial_DIN0207_L6.3mm_D2.5mm_P10.16mm_Horizontal -> Resistor_SMD:R_0603_1608Metric; now not fitted
- R11: value 10k -> 1k; footprint Resistor_THT:R_Axial_DIN0207_L6.3mm_D2.5mm_P10.16mm_Horizontal -> Resistor_SMD:R_0603_1608Metric
- R12: renamed from R14; footprint Resistor_THT:R_Axial_DIN0207_L6.3mm_D2.5mm_P10.16mm_Horizontal -> Resistor_SMD:R_0603_1608Metric
- R13: renamed from R12; value 51 -> 1k; footprint Resistor_THT:R_Axial_DIN0207_L6.3mm_D2.5mm_P10.16mm_Horizontal -> Resistor_SMD:R_0603_1608Metric
- R14: renamed from R13; footprint Resistor_THT:R_Axial_DIN0207_L6.3mm_D2.5mm_P10.16mm_Horizontal -> Resistor_SMD:R_0603_1608Metric
- R3: value 1k -> 5.1k
- R9: value 1.5k -> 1k; footprint Resistor_THT:R_Axial_DIN0207_L6.3mm_D2.5mm_P10.16mm_Horizontal -> Resistor_SMD:R_0603_1608Metric
- SW1: value TVGP01-G73BB -> RUN; footprint Button_Switch_THT:SW_PUSH-12mm -> AM_Switch:TVBP06-B043Cx-B; Akizuki_code (none) -> 108074; now not fitted
- U6: renamed from U3; Akizuki_code (none) -> 114063
- U7: renamed from U4; Akizuki_code (none) -> 116585
- renumbered D2 to D3, R1 to R27, R2 to R28, R4 to R37, R5 to R38, R6 to R39, R7 to R42
Connections:
- net +5V: now also C2.1, J5.1 (Pin_1), C1.1, C19.1, C20.1, C21.1, C22.1, C23.1, C24.1, J6.1 (Pin_1), JP1.2 (B), R16.2, R17.1, R18.1, R2.2, R24.2, R26.1, R35.2, R43.2, R44.2, R45.2, R6.1, U1.5 (Vin), U10.8 (VCC), U10.8 (VCC), U11.8 (VCC), U11.8 (VCC), U4.8 (VCC), U4.8 (VCC), U5.3 (VDD), U9.8 (VCC), U9.8 (VCC); no longer C16.1, C3.2, R11.1, R9.1, SW1.1
- net ADC_SCL: now also U2.30 (GPIO19)
- net ADC_SDA: now also U2.29 (GPIO18)
- net GND: now also C17.1, C3.2, R3.2, SW1.1, U6.4 (GND), C1.2, C10.2, C11.2, C12.2, C13.2, C14.2, C15.2, C19.2, C20.2, C21.2, C22.2, C23.2, C24.2, C4.2, C5.1, C6.2, C7.2, C8.2, C9.2, J4.3 (Pin_3), J8.4 (Pin_4), JP2.1 (A), Q1.2 (S), R1.2, R29.1, R30.1, R32.1, R40.1, R41.1, R8.1, RV1.1, RV1.2, RV2.2, RV2.3, RV3.2, RV3.3, RV4.1, RV4.2, SW2.1, U1.2 (GND), U10.4 (GND), U10.4 (GND), U11.4 (GND), U11.4 (GND), U2.19 (TESTEN), U2.57 (GND), U3.4 (GND), U3.9 (EPAD), U4.4 (GND), U4.4 (GND), U5.2 (VSS), U8.2 (Anode), U9.4 (GND), U9.4 (GND), Y1.2, Y1.4; no longer C3.1, J5.2 (Pin_2), R10.2
- net LOAD_ENABLE: now also U2.37 (GPIO25)
- net SHUNT_SELECT1: now also U2.35 (GPIO23)
- net SHUNT_SELECT2: now also U2.34 (GPIO22)
- net VAA: now also R26.2, R31.2, U5.6 (Vref), U8.3 (Cathod); no longer R3.1
- net Vconst_ENABLE: now also U2.36 (GPIO24)
- net Vofs: now also J8.3 (Pin_3), U11.1, U11.2; no longer J5.1 (Pin_1), U6.1, U6.2
- net ROM_SS: now reaches R11.2
- net ROM_SS: now also R10.1, SW2.2, U2.56 (QSPI_SS); no longer C17.1
- net Vmeas: now reaches U7.1 (Vin+)
- net Vmeas: now also J8.1 (Pin_1), TP7.1
- net at U6.5: now also R25.1, R29.2
- net DAC_SCK renamed LED_Gate1
- net LED_Gate1: now also U2.27 (GPIO16)
- net TEMPERATURE: no longer names the net of U6.6
- net TEMPERATURE: now also R21.2, R23.2; no longer U6.7
- net UART_RTS: no longer names the net of D1.2 (A)
- net UART_RTS: now also J2.A4 (VBUS), J2.A9 (VBUS), J2.B4 (VBUS), J2.B9 (VBUS)
- new net: C17.2, R9.1, Y1.1
- new net: C5.2, U2.20 (XIN), Y1.3
- new net: C25.1, R15.1, R19.2, U4.2
- new net: D2.1 (K), Q1.3 (D)
- new net: D2.2 (A), R6.2
- new net: R31.1, R32.2, U8.1 (REF)
- new net: R44.1, RV3.1, U10.5
- new net: R16.1, RV1.3, U4.5
- new net: R45.1, RV4.3, U11.5
- new net: R33.2, R34.2, U9.6
- new net: J6.2 (Pin_2), R35.1, R41.2, U9.3
- new net: D1.1 (K), JP1.1 (A)
- new net: R43.1, RV2.1, U10.3
- new net: R20.2, R22.2, U4.3
- new net: R20.1, U5.1 (VOUT)
- new net: SW1.2, U2.26 (RUN)
- new net: J5.2 (Pin_2), R24.1, R30.2, U6.3
- new net: R36.1, R40.2, U9.5
- new net: R36.2, U9.1, U9.2
- new net: R11.1, U3.1 (~{CS})
- new net: J2.B5 (CC2), R3.1
- new net: J1.1 (Pin_1), U2.2 (GPIO0)
- new net: J1.10 (Pin_10), U2.12 (GPIO9)
- new net: J1.11 (Pin_11), U2.13 (GPIO10)
- new net: J1.12 (Pin_12), U2.14 (GPIO11)
- new net: J1.13 (Pin_13), U2.15 (GPIO12)
- new net: J1.14 (Pin_14), U2.16 (GPIO13)
- new net: J1.15 (Pin_15), U2.17 (GPIO14)
- new net: J1.16 (Pin_16), U2.18 (GPIO15)
- new net: J1.2 (Pin_2), U2.3 (GPIO1)
- new net: J1.3 (Pin_3), U2.4 (GPIO2)
- new net: J1.4 (Pin_4), U2.5 (GPIO3)
- new net: J1.5 (Pin_5), U2.6 (GPIO4)
- new net: J1.6 (Pin_6), U2.7 (GPIO5)
- new net: J1.7 (Pin_7), U2.8 (GPIO6)
- new net: J1.8 (Pin_8), U2.9 (GPIO7)
- new net: J1.9 (Pin_9), U2.11 (GPIO8)
- new net: R9.2, U2.21 (XOUT)
- new net: R2.1, U1.1 (Ctrl)
- new net: C4.1, U1.3 (Cap)
- new net: J2.A1 (GND), J2.A12 (GND), J2.B1 (GND), J2.B12 (GND), JP2.2 (B)
- new net: R25.2, U6.1, U6.2
- new net: Q1.1 (G), R7.2, R8.2
- new net: J2.A5 (CC1), R1.1
- new net +1V1: C14.1, C15.1, C16.1, U2.23 (DVDD), U2.45 (VREG_VOUT), U2.50 (DVDD)
- new net +3V3: C10.1, C11.1, C12.1, C13.1, C3.1, C6.1, C7.1, C8.1, C9.1, J4.1 (Pin_1), R10.2, U1.4 (Vout), U2.1 (IOVDD), U2.10 (IOVDD), U2.22 (IOVDD), U2.33 (IOVDD), U2.42 (IOVDD), U2.43 (ADC_AVDD), U2.44 (VREG_IN), U2.48 (USB_VDD), U2.49 (IOVDD), U3.8 (VCC)
- new net DAC_SCL: R18.2, U2.32 (GPIO21), U5.5 (SCL)
- new net DAC_SDA: R17.2, U2.31 (GPIO20), U5.4 (SDA)
- new net LED_Gate2: R7.1, U2.28 (GPIO17)
- new net MOS_TEMP: R33.1, TP8.1, U2.40 (GPIO28_ADC2), U9.7
- new net RES_TEMP: R21.1, TP6.1, U2.41 (GPIO29_ADC3), U6.7
- new net ROM_CLK: U2.52 (QSPI_SCLK), U3.6 (CLK)
- new net ROM_IO0: U2.53 (QSPI_SD0), U3.5 (DI/IO_{0})
- new net ROM_IO1: U2.55 (QSPI_SD1), U3.2 (DO/IO_{1})
- new net ROM_IO2: U2.54 (QSPI_SD2), U3.3 (~{WP}/IO_{2})
- new net ROM_IO3: U2.51 (QSPI_SD3), U3.7 (~{HOLD}/~{RESET}/IO_{3})
- new net SWCLK: J4.2 (Pin_2), U2.24 (SWCLK)
- new net SWD: J4.4 (Pin_4), U2.25 (SWD)
- new net T_ofs1: R23.1, U10.1, U10.2
- new net T_ofs2: R34.1, U10.6, U10.7
- new net USB+: J2.A6 (D+), J2.B6 (D+), R5.1
- new net USB-: J2.A7 (D-), J2.B7 (D-), R4.1
- new net USB_D+: R5.2, U2.47 (USB_DP)
- new net USB_D-: R4.2, U2.46 (USB_DM)
- new net Vofs1: R22.1, U11.3, U11.6, U11.7
- new net Vref: C25.2, J8.2 (Pin_2), R15.2, TP5.1, U4.1
- new net VrefCMP: R19.1, U4.6, U4.7
- no-connect marks 1 -> 3
Other:
- note added: "ADC, DAC"
- note added: "OPAMP"
- note added: "RP2040"
- moved on the sheet: C26, D3, J5, J7, J9, Q2, R12, R13, R14, R27, R28, R37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
